Commit message: feat: expose vlp gpu ray

File: src/jackal_description/urdf/accessories/vlp16_mount.urdf.xacro (robot description, xacro)
@@ -1,5 +1,5 @@
 <robot xmlns:xacro="http://wiki.ros.org/xacro">
   <xacro:include filename="$(find velodyne_description)/urdf/VLP-16.urdf.xacro" />
-  <xacro:macro name="vlp16_mount" params="prefix parent_link topic tower height:=0.1 *origin">
+  <xacro:macro name="vlp16_mount" params="prefix parent_link topic tower height:=0.1 *origin gpu">
     <xacro:if value="${tower}">
       <link name="${prefix}_vlp16_mount" />
@@ -87,10 +87,12 @@
         <origin xyz="0 0 ${height}" rpy="0 0 0" />
       </joint>
-      <xacro:VLP-16 parent="${prefix}_vlp16_plate" topic="${topic}">
+      <xacro:VLP-16 parent="${prefix}_vlp16_plate" topic="${topic}" gpu="${gpu}">
+    <!-- <xacro:VLP-16 parent="${prefix}_vlp16_plate" topic="${topic}"> -->
         <origin xyz="0 0 0" rpy="0 0 0" />
       </xacro:VLP-16>
     </xacro:if>
     <xacro:unless value="${tower}">
-      <xacro:VLP-16 parent="${parent_link}" topic="${topic}">
+      <xacro:VLP-16 parent="${parent_link}" topic="${topic}" gpu="${gpu}">
+    <!-- <xacro:VLP-16 parent="${parent_link}" topic="${topic}"> -->
         <xacro:insert_block name="origin" />
       </xacro:VLP-16>
