Commit message: feat: enable gpu ray

File: src/jackal_description/urdf/accessories.urdf.xacro (robot description, xacro)
@@ -176,7 +176,8 @@
     <xacro:property name="parent" value="$(optenv JACKAL_LASER_3D_PARENT ${mount}_mount)" />
     <xacro:property name="lidar_3d_model" value="$(optenv JACKAL_LASER_3D_MODEL vlp16)" />
+    <xacro:property name="gpu" value="$(optenv JACKAL_LASER_3D_GPU 1)" />
     <!-- Velodyne VLP16 -->
     <xacro:if value="${lidar_3d_model == 'vlp16'}">
-      <xacro:vlp16_mount topic="${topic}" tower="${tower}" prefix="${prefix}" parent_link="${parent}" >
+      <xacro:vlp16_mount topic="${topic}" tower="${tower}" prefix="${prefix}" parent_link="${parent}" gpu="${gpu}">
         <origin xyz="$(optenv JACKAL_LASER_3D_OFFSET 0 0 0)" rpy="$(optenv JACKAL_LASER_3D_RPY 0 0 0)" />
       </xacro:vlp16_mount>

Commit message: feat: expose velodyne min range

File: src/jackal_description/urdf/accessories.urdf.xacro (robot description, xacro)
@@ -177,7 +177,9 @@
     <xacro:property name="lidar_3d_model" value="$(optenv JACKAL_LASER_3D_MODEL vlp16)" />
     <xacro:property name="gpu" value="$(optenv JACKAL_LASER_3D_GPU 1)" />
+    <xacro:property name="collision_range" value="$(optenv JACKAL_LASER_3D_COLLISION_RANGE 0.15)" />
+    <xacro:property name="min_range" value="$(optenv JACKAL_LASER_3D_MIN_RANGE 0.5)" />
     <!-- Velodyne VLP16 -->
     <xacro:if value="${lidar_3d_model == 'vlp16'}">
-      <xacro:vlp16_mount topic="${topic}" tower="${tower}" prefix="${prefix}" parent_link="${parent}" gpu="${gpu}">
+      <xacro:vlp16_mount topic="${topic}" tower="${tower}" prefix="${prefix}" parent_link="${parent}" gpu="${gpu}" collision_range="${collision_range}" min_range="${min_range}">
         <origin xyz="$(optenv JACKAL_LASER_3D_OFFSET 0 0 0)" rpy="$(optenv JACKAL_LASER_3D_RPY 0 0 0)" />
       </xacro:vlp16_mount>

File: src/jackal_description/urdf/accessories/vlp16_mount.urdf.xacro (robot description, xacro)
@@ -1,5 +1,5 @@
 <robot xmlns:xacro="http://wiki.ros.org/xacro">
   <xacro:include filename="$(find velodyne_description)/urdf/VLP-16.urdf.xacro" />
-  <xacro:macro name="vlp16_mount" params="prefix parent_link topic tower height:=0.1 *origin gpu">
+  <xacro:macro name="vlp16_mount" params="prefix parent_link topic tower height:=0.1 *origin gpu collision_range:=0.15 min_range:=0.5">
     <xacro:if value="${tower}">
       <link name="${prefix}_vlp16_mount" />
@@ -87,5 +87,5 @@
         <origin xyz="0 0 ${height}" rpy="0 0 0" />
       </joint>
-      <xacro:VLP-16 parent="${prefix}_vlp16_plate" topic="${topic}" gpu="${gpu}">
+      <xacro:VLP-16 parent="${prefix}_vlp16_plate" topic="${topic}" gpu="${gpu}" collision_range="${collision_range}" min_range="${min_range}">
     <!-- <xacro:VLP-16 parent="${prefix}_vlp16_plate" topic="${topic}"> -->
         <origin xyz="0 0 0" rpy="0 0 0" />
@@ -93,5 +93,5 @@
     </xacro:if>
     <xacro:unless value="${tower}">
-      <xacro:VLP-16 parent="${parent_link}" topic="${topic}" gpu="${gpu}">
+      <xacro:VLP-16 parent="${parent_link}" topic="${topic}" gpu="${gpu}" collision_range="${collision_range}" min_range="${min_range}">
     <!-- <xacro:VLP-16 parent="${parent_link}" topic="${topic}"> -->
         <xacro:insert_block name="origin" />
